File: xc7z010_ddr3/ddr3-sodimm.sch (KiCad schematic (older format))
At the start: 12 parts, among them J1 SODIMM-204

Commit message: init
Parts:
- U1: renamed from U?; symbol xc7z010_ddr3-rescue:XC7Z010-CLG400-mybays_fpga_cpld -> mybays_fpga_cpld:XC7Z010-CLG400
- gave numbers to parts that had none: 10
Changed lines of the file:
@@
 DDR_DQS_N3
 $Comp
-L Device:R_US R?
+L Device:R_US R1
 U 1 1 60571F65
 P 5500 7150
-F 0 "R?" V 5450 7050 50  0000 C CNN
+F 0 "R1" V 5450 7050 50  0000 C CNN
 F 1 "80.5" V 5450 7300 50  0000 C CNN
 F 2 "Resistor_SMD:R_0402_1005Metric" V 5540 7140 50  0001 C CNN
@@
 $EndComp
 $Comp
-L Device:R_US R?
+L Device:R_US R2
 U 1 1 6057348E
 P 5500 7250
-F 0 "R?" V 5450 7150 50  0000 C CNN
+F 0 "R2" V 5450 7150 50  0000 C CNN
 F 1 "80.5" V 5450 7400 50  0000 C CNN
 F 2 "Resistor_SMD:R_0402_1005Metric" V 5540 7240 50  0001 C CNN
@@
 	5200 7250 5350 7250
 $Comp
-L power:GND #PWR?
+L power:GND #PWR0101
 U 1 1 60575495
 P 5800 7100
-F 0 "#PWR?" H 5800 6850 50  0001 C CNN
+F 0 "#PWR0101" H 5800 6850 50  0001 C CNN
 F 1 "GND" H 5805 6927 50  0000 C CNN
 F 2 "" H 5800 7100 50  0001 C CNN
@@
 	5800 7150 5800 7100
 $Comp
-L power:+1V35 #PWR?
+L power:+1V35 #PWR0102
 U 1 1 60577607
 P 3900 8850
-F 0 "#PWR?" H 3900 8700 50  0001 C CNN
+F 0 "#PWR0102" H 3900 8700 50  0001 C CNN
 F 1 "+1V35" H 3915 9023 50  0000 C CNN
 F 2 "" H 3900 8850 50  0001 C CNN
@@
 VCC_DDR
 $Comp
-L Device:C C?
+L Device:C C1
 U 1 1 6057C3AE
 P 5400 7900
-F 0 "C?" H 5500 7800 50  0000 R CNN
+F 0 "C1" H 5500 7800 50  0000 R CNN
 F 1 "100n" H 5550 8000 50  0000 R CNN
 F 2 "Capacitor_SMD:C_0402_1005Metric" H 5438 7750 50  0001 C CNN
@@
 $EndComp
 $Comp
-L Device:C C?
+L Device:C C2
 U 1 1 6057F542
 P 5400 8300
-F 0 "C?" H 5500 8200 50  0000 R CNN
+F 0 "C2" H 5500 8200 50  0000 R CNN
 F 1 "100n" H 5550 8400 50  0000 R CNN
 F 2 "Capacitor_SMD:C_0402_1005Metric" H 5438 8150 50  0001 C CNN
@@
 $EndComp
 $Comp
-L xc7z010_ddr3-rescue:XC7Z010-CLG400-mybays_fpga_cpld U?
+L mybays_fpga_cpld:XC7Z010-CLG400 U?
 U 8 1 60535F38
 P 3300 5400
 AR Path="/60535F38" Ref="U?"  Part="8"
 AR Path="/6036CA45/60535F38" Ref="U?"  Part="8"
-AR Path="/603605FC/60535F38" Ref="U?"  Part="8"
-F 0 "U?" H 3300 8317 50  0000 C CNN
+AR Path="/603605FC/60535F38" Ref="U1"  Part="8"
+F 0 "U1" H 3300 8317 50  0000 C CNN
 F 1 "XC7Z010-CLG400" H 3300 8226 50  0000 C CNN
 F 2 "mybays_fpga_cpld:CLG400-0.8" H 1700 2750 50  0001 C CNN
@@
 Connection ~ 5400 8100
 $Comp
-L Device:R_US R?
+L Device:R_US R3
 U 1 1 60582A40
 P 5600 7900
-F 0 "R?" V 5550 7800 50  0000 C CNN
+F 0 "R3" V 5550 7800 50  0000 C CNN
 F 1 "1.2k" V 5550 8050 50  0000 C CNN
 F 2 "Resistor_SMD:R_0402_1005Metric" V 5640 7890 50  0001 C CNN
@@
 $EndComp
 $Comp
-L Device:R_US R?
+L Device:R_US R4
 U 1 1 60583F2D
 P 5600 8300
-F 0 "R?" V 5550 8200 50  0000 C CNN
+F 0 "R4" V 5550 8200 50  0000 C CNN
 F 1 "1.2k" V 5550 8450 50  0000 C CNN
 F 2 "Resistor_SMD:R_0402_1005Metric" V 5640 8290 50  0001 C CNN
@@
 	5600 8100 5600 8150
 $Comp
-L power:GND #PWR?
+L power:GND #PWR0103
 U 1 1 60586F9F
 P 5500 8550
-F 0 "#PWR?" H 5500 8300 50  0001 C CNN
+F 0 "#PWR0103" H 5500 8300 50  0001 C CNN
 F 1 "GND" H 5505 8377 50  0000 C CNN
 F 2 "" H 5500 8550 50  0001 C CNN
@@
 	5600 7650 5600 7750
 $Comp
-L Device:C C?
+L Device:C C3
 U 1 1 6058E880
 P 6000 7900
-F 0 "C?" H 6100 7800 50  0000 R CNN
+F 0 "C3" H 6100 7800 50  0000 R CNN
 F 1 "100n" H 6150 8000 50  0000 R CNN
 F 2 "Capacitor_SMD:C_0402_1005Metric" H 6038 7750 50  0001 C CNN
@@
 $EndComp
 $Comp
-L Device:C C?
+L Device:C C4
 U 1 1 6058E886
 P 6000 8300
-F 0 "C?" H 6100 8200 50  0000 R CNN
+F 0 "C4" H 6100 8200 50  0000 R CNN
 F 1 "100n" H 6150 8400 50  0000 R CNN
 F 2 "Capacitor_SMD:C_0402_1005Metric" H 6038 8150 50  0001 C CNN
@@
 Connection ~ 6000 8100
 $Comp
-L Device:R_US R?
+L Device:R_US R5
 U 1 1 6058E890
 P 6200 7900
-F 0 "R?" V 6150 7800 50  0000 C CNN
+F 0 "R5" V 6150 7800 50  0000 C CNN
 F 1 "1.2k" V 6150 8050 50  0000 C CNN
 F 2 "Resistor_SMD:R_0402_1005Metric" V 6240 7890 50  0001 C CNN
@@
 $EndComp
 $Comp
-L Device:R_US R?
+L Device:R_US R6
 U 1 1 6058E896
 P 6200 8300
-F 0 "R?" V 6150 8200 50  0000 C CNN
+F 0 "R6" V 6150 8200 50  0000 C CNN
 F 1 "1.2k" V 6150 8450 50  0000 C CNN
 F 2 "Resistor_SMD:R_0402_1005Metric" V 6240 8290 50  0001 C CNN
@@
 	6200 8100 6200 8150
 $Comp
-L power:GND #PWR?
+L power:GND #PWR0104
 U 1 1 6058E8A0
 P 6100 8550
-F 0 "#PWR?" H 6100 8300 50  0001 C CNN
+F 0 "#PWR0104" H 6100 8300 50  0001 C CNN
 F 1 "GND" H 6105 8377 50  0000 C CNN
 F 2 "" H 6100 8550 50  0001 C CNN

Commit message: 202101212
Connections:
- net +1V35: now also J1.100, J1.105, J1.106, J1.111, J1.112, J1.117, J1.118, J1.123, J1.124, J1.75, J1.76, J1.81, J1.82, J1.87, J1.88, J1.93, J1.94, J1.99
- net DDR_CAS: now also J1.115
- net DDR_RAS: now also J1.110
- net DDR_WE: now also J1.113
- net GND: now also J1.127, J1.13, J1.133, J1.134, J1.138, J1.139, J1.14, J1.144, J1.145, J1.150, J1.151, J1.155, J1.156, J1.161, J1.162, J1.167, J1.168, J1.172, J1.173, J1.178, J1.179, J1.184, J1.185, J1.189, J1.19, J1.190, J1.195, J1.196, J1.2, J1.20, J1.25, J1.26, J1.3, J1.31, J1.32, J1.37, J1.38, J1.43, J1.44, J1.48, J1.49, J1.54, J1.55, J1.60, J1.61, J1.65, J1.66, J1.71, J1.72, J1.8, J1.9
- net DDR_CK0_N: now reaches J1.101
- net DDR_CK1_P: now reaches J1.102
- net DDR_CK0_P: now reaches J1.103
- net DDR_CK1_N: now reaches J1.104
- net DDR_S0: now reaches J1.114
- net DDR_ODT1: now reaches J1.120
- net DDR_S1: now reaches J1.121
- net DDR_VREFCA: now reaches J1.126
- net DDR_SS: now reaches J1.128
- net DDR_DQS_N4: now reaches J1.135
- net DDR_DQS_P4: now reaches J1.137
- net DDR_DQS_N5: now reaches J1.152
- net DDR_DM5: now reaches J1.153
- net DDR_DQS_P5: now reaches J1.154
- net DDR_DQS_N6: now reaches J1.169
- net DDR_DM6: now reaches J1.170
- net DDR_DQS_P6: now reaches J1.171
- net DDR_DQS_N7: now reaches J1.186
- net DDR_DM7: now reaches J1.187
- net DDR_DQS_P7: now reaches J1.188
- net DDR_SA0: now reaches J1.197
- net DDR_EVENT: now reaches J1.198
- net DDR_VDD_SPD: now reaches J1.199
- net DDR_SDA: now reaches J1.200
- net DDR_SA1: now reaches J1.201
- net DDR_SCL: now reaches J1.202
- net DDR_VTT: now reaches J1.203
- net DDR_VTT: now also J1.204
- net DDR_CKE0: now reaches J1.73
- net DDR_CKE1: now reaches J1.74
- no-connect marks 0 -> 4
